File: projects/pinion/hardware/pinion-main/io-mcu.kicad_sch (KiCad schematic)
At the start: 0 parts

Commit message: [pinion] added mcu, mpu and external library
Parts:
- added U2: STM32F103C8Tx, Package_QFP:LQFP-48_7x7mm_P0.5mm, symbol MCU_ST_STM32F1:STM32F103C8Tx
Connections:
- new net: U2.23 (VSS), U2.35 (VSS), U2.47 (VSS)
Changed lines of the file:
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@@
 	(generator_version "10.0")
 	(paper "A4")
+	(symbol
+		(lib_id "MCU_ST_STM32F1:STM32F103C8Tx")
+		(at 144.78 91.44 0)
+		(unit 1)
+		(body_style 1)
+		(exclude_from_sim no)
+		(in_bom yes)
+		(on_board yes)
+		(in_pos_files yes)
+		(dnp no)
+		(fields_autoplaced yes)
+		(property "Reference" "U2"
+			(at 149.4633 132.08 0)
+			(show_name no)
+			(do_not_autoplace no)
+			(effects
+				(font
+					(size 1.27 1.27)
+				)
+				(justify left)
+			)
+		)
+		(property "Value" "STM32F103C8Tx"
+			(at 149.4633 134.62 0)
+			(show_name no)
+			(do_not_autoplace no)
+			(effects
+				(font
+					(size 1.27 1.27)
+				)
+				(justify left)
+			)
+		)
+		(property "Footprint" "Package_QFP:LQFP-48_7x7mm_P0.5mm"
+			(at 129.54 129.54 0)
+			(hide yes)
+			(show_name no)
+			(do_not_autoplace no)
+			(effects
+				(font
+					(size 1.27 1.27)
+				)
+				(justify right)
+			)
+		)
+		(property "Datasheet" "https://www.st.com/resource/en/datasheet/stm32f103c8.pdf"
+			(at 144.78 91.44 0)
+			(hide yes)
+			(show_name no)
+			(do_not_autoplace no)
+			(effects
+				(font
+					(size 1.27 1.27)
+				)
+			)
+		)
+		(property "Description" "STMicroelectronics Arm Cortex-M3 MCU, 64KB flash, 20KB RAM, 72 MHz, 2.0-3.6V, 37 GPIO, LQFP48"
+			(at 144.78 91.44 0)
+			(hide yes)
+			(show_name no)
+			(do_not_autoplace no)
+			(effects
+				(font
+					(size 1.27 1.27)
+				)
+			)
+		)
+		(pin "33"
+		)
+		(pin "32"
+		)
+		(pin "27"
+		)
+		(pin "31"
+		)
+		(pin "30"
+		)
+		(pin "28"
+		)
+		(pin "29"
+		)
+		(pin "5"
+		)
+		(pin "6"
+		)
+		(pin "4"
+		)
+		(pin "7"
+		)
+		(pin "3"
+		)
+		(pin "2"
+		)
+		(pin "1"
+		)
+		(pin "9"
+		)
+		(pin "35"
+		)
+		(pin "37"
+		)
+		(pin "36"
+		)
+		(pin "34"
+		)
+		(pin "11"
+		)
+		(pin "10"
+		)
+		(pin "12"
+		)
+		(pin "14"
+		)
+		(pin "13"
+		)
+		(pin "15"
+		)
+		(pin "20"
+		)
+		(pin "18"
+		)
+		(pin "17"
+		)
+		(pin "19"
+		)
+		(pin "16"
+		)
+		(pin "46"
+		)
+		(pin "47"
+		)
+		(pin "48"
+		)
+		(pin "8"
+		)
+		(pin "26"
+		)
+		(pin "25"
+		)
+		(pin "24"
+		)
+		(pin "22"
+		)
+		(pin "23"
+		)
+		(pin "42"
+		)
+		(pin "21"
+		)
+		(pin "44"
+		)
+		(pin "45"
+		)
+		(pin "43"
+		)
+		(pin "40"
+		)
+		(pin "38"
+		)
+		(pin "41"
+		)
+		(pin "39"
+		)
+		(instances
+			(project "pinion-main"
+				(path "/6c7907f5-5439-4f54-a5a2-0a7e85489635/e3d61feb-6226-49e9-91f2-6966c39438aa/2e8c24c6-430a-4c2a-bf9a-526269dfdd68"
+					(reference "U2")
+					(unit 1)
+				)
+			)
+		)
+	)
 )
