File: projects/pinion/hardware/pinion-main/soc.kicad_sch (KiCad schematic)
At the start: 0 parts

Commit message: [pinion] added mcu, mpu and external library
Parts:
- added U3: XAM62L32AOGHAANB, Texas_Instruments:FCCSP373_11P9X11P9_TEX, symbol lib:XAM62L32AOGHAANB
Connections:
- new net: U3.A1 (VSS), U3.A10 (VSS), U3.A13 (VSS), U3.A16 (VSS), U3.A19 (VSS), U3.A2 (VSS), U3.A22 (VSS), U3.A23 (VSS), U3.A4 (VSS), U3.AA20 (VSS), U3.AA4 (VSS), U3.AB1 (VSS), U3.AB21 (VSS), U3.AB23 (VSS), U3.AB7 (VSS), U3.AC1 (VSS), U3.AC11 (VSS), U3.AC14 (VSS), U3.AC19 (VSS), U3.AC2 (VSS), U3.AC22 (VSS), U3.AC23 (VSS), U3.B1 (VSS), U3.B17 (VSS), U3.B20 (VSS), U3.B23 (VSS), U3.B5 (VSS), U3.C12 (VSS), U3.C18 (VSS), U3.D1 (VSS), U3.E10 (VSS), U3.E14 (VSS), U3.E15 (VSS), U3.E2 (VSS), U3.E6 (VSS), U3.E8 (VSS), U3.E9 (VSS), U3.F18 (VSS), U3.F5 (VSS), U3.F6 (VSS), U3.G12 (VSS), U3.G15 (VSS), U3.G16 (VSS), U3.G17 (VSS), U3.G7 (VSS), U3.G8 (VSS), U3.G9 (VSS), U3.H1 (VSS), U3.H14 (VSS), U3.H17 (VSS), U3.H7 (VSS), U3.K15 (VSS), U3.K8 (VSS), U3.K9 (VSS), U3.L13 (VSS), U3.L16 (VSS), U3.L18 (VSS), U3.L7 (VSS), U3.L9 (VSS), U3.M1 (VSS), U3.M12 (VSS), U3.N11 (VSS), U3.N13 (VSS), U3.N16 (VSS), U3.N7 (VSS), U3.N9 (VSS), U3.P15 (VSS), U3.P9 (VSS), U3.R1 (VSS), U3.R13 (VSS), U3.R15 (VSS), U3.R8 (VSS), U3.T19 (VSS), U3.T2 (VSS), U3.T7 (VSS), U3.T8 (VSS), U3.U10 (VSS), U3.U13 (VSS), U3.U14 (VSS), U3.U15 (VSS), U3.U17 (VSS), U3.U20 (VSS), U3.U7 (VSS), U3.U8 (VSS), U3.V18 (VSS), U3.V19 (VSS), U3.V3 (VSS), U3.W10 (VSS), U3.W12 (VSS), U3.W14 (VSS), U3.W15 (VSS), U3.W16 (VSS), U3.W18 (VSS), U3.W9 (VSS), U3.Y1 (VSS), U3.Y20 (VSS), U3.Y21 (VSS)
- new net: U3.G10 (VDDSHV1), U3.H10 (VDDSHV1)
- new net: U3.J11 (VDD_CORE), U3.J13 (VDD_CORE), U3.J15 (VDD_CORE), U3.J9 (VDD_CORE), U3.K10 (VDD_CORE), U3.K14 (VDD_CORE), U3.L15 (VDD_CORE), U3.M14 (VDD_CORE), U3.N15 (VDD_CORE), U3.P10 (VDD_CORE), U3.P12 (VDD_CORE), U3.P14 (VDD_CORE), U3.R11 (VDD_CORE), U3.R9 (VDD_CORE)
- new net: U3.J16 (VDDSHV0), U3.L17 (VDDSHV0)
- new net: U3.L8 (VDDS_DDR), U3.M7 (VDDS_DDR), U3.M8 (VDDS_DDR), U3.N8 (VDDS_DDR), U3.P8 (VDDS_DDR)
