File: projects/pinion/hardware/pinion-main/fmu-power.kicad_sch (KiCad schematic)
At the start: 0 parts

Commit message: [pinion] 3v3 power for sys and fmu
Parts:
- added C15: 100n, Capacitor_SMD:C_0402_1005Metric, symbol Device:C_Small
- added C16: 47p, Capacitor_SMD:C_0402_1005Metric, symbol Device:C_Small
- added C17, C18: 10u, Capacitor_SMD:C_0805_2012Metric, symbol Device:C_Small
- added L1: 4.7u, Inductor_SMD:L_1008_2520Metric, symbol Device:L_Small
- added R23, R25: 100k, Resistor_SMD:R_0402_1005Metric, symbol Device:R_Small_US
- added R24: 22.1k, Resistor_SMD:R_0402_1005Metric, symbol Device:R_Small_US
- added TP1: TestPoint, symbol Connector:TestPoint
- added U13: SY8120IABC, Package_TO_SOT_SMD:SOT-23-6, symbol Regulator_Switching:LGS5116B
Connections:
- new net: C15.1, U13.1 (BST)
- new net: C15.2, L1.1, U13.6 (SW)
- new net: C16.2, R23.2, R24.1, U13.3 (FB)
- new net: R25.2, U13.4 (EN)
- new net +5V: C18.1, R25.1, U13.5 (VIN)
- new net FMU_VDD_3V3: C16.1, C17.1, L1.2, R23.1, TP1.1
- new net GND: C17.2, C18.2, R24.2, U13.2 (GND)

Commit message: [pinion] mcu basic schematic in
Parts:
- added C23, C24, C25: 10u, Capacitor_SMD:C_0805_2012Metric, symbol Device:C_Small
- added C26, C27: 150u, Capacitor_SMD:CP_Elec_6.3x5.7, symbol Device:C_Polarized_Small_US
- added C28, C29: 1u, Capacitor_SMD:C_0603_1608Metric, symbol Device:C_Small
- added FB1: 200, Inductor_SMD:L_0603_1608Metric, symbol Device:FerriteBead_Small
- added R29, R30, R31, R32, R33, R34, R35, R36: 100k, Resistor_SMD:R_0402_1005Metric, symbol Device:R_Small_US
- added TP10, TP11, TP3, TP4, TP5, TP6, TP7, TP8, TP9: TestPoint, TestPoint:TestPoint_Pad_D1.0mm, symbol Connector:TestPoint
- added U15, U18: SY6288CAAC, Package_TO_SOT_SMD:SOT-23-5, symbol Power_Management:AP22818AKEWT
- added U16, U17: SY6288AAAC, Package_TO_SOT_SMD:SOT-23-5, symbol Power_Management:AP22816AKEWT
- TP1: footprint (none) -> TestPoint:TestPoint_Pad_D1.0mm
Connections:
- net +5V: now also C28.2, C29.2, U15.5 (IN), U18.5 (IN)
- net FMU_VDD_3V3: now also FB1.1, R30.2, R32.2, R34.2, R36.2, U16.5 (IN), U17.5 (IN)
- net GND: now also C23.2, C24.2, C25.2, C26.2, C27.2, C28.1, C29.1, R29.2, R31.2, R33.2, R35.2, U15.2 (GND), U16.2 (GND), U17.2 (GND), U18.2 (GND)
- new net FMU_VDDA_3V3: C23.1, FB1.2, TP3.1
- new net FMU_VDD_3V3_SENSORS: C24.1, TP4.1, U16.1 (OUT)
- new net FMU_VDD_3V3_SENSORS_EN: R29.1, U16.4 (EN)
- new net FMU_VDD_3V3_SENSORS_FLT: R30.1, TP5.1, U16.3 (~{FLG})
- new net FMU_VDD_5V_HIPWR: C27.1, TP10.1, U18.1 (OUT)
- new net FMU_VDD_5V_HIPWR_EN: R35.1, U18.4 (EN)
- new net FMU_VDD_5V_HIPWR_FLT: R36.1, TP11.1, U18.3 (~{FLG})
- new net FMU_VDD_5V_PERIPH: C26.1, TP8.1, U15.1 (OUT)
- new net FMU_VDD_5V_PERIPH_EN: R33.1, U15.4 (EN)
- new net FMU_VDD_5V_PERIPH_FLT: R34.1, TP9.1, U15.3 (~{FLG})
- new net IO_VDD_3V3_SPEKTRUM: C25.1, TP6.1, U17.1 (OUT)
- new net IO_VDD_3V3_SPEKTRUM_EN: R31.1, U17.4 (EN)
- new net IO_VDD_3V3_SPEKTRUM_FLT: R32.1, TP7.1, U17.3 (~{FLG})
Other:
- note added: "POWER SWITCH SIGNAL POLARITY *_EN Active high: high turns the rail on. 100k pull-down keeps the rail off during reset. *_FLT Active low, open drain: low means overcurrent or overtemperature. 100k pull-up to FMU_VDD_3V3."
- moved on the sheet: C15, C16, C17, C18, L1, R23, R24, R25, TP1, U13
