File: projects/pinion/hardware/pinion-main/fmu-connectors.kicad_sch (KiCad schematic)
At the start: 0 parts

Commit message: [pinion] fmu connectors and esd protection
Parts:
- added C55: 100n, Capacitor_SMD:C_0402_1005Metric, symbol Device:C_Small
- added C56, C57: 1u, Capacitor_SMD:C_0402_1005Metric, symbol Device:C_Small
- added D11, D12: NUP2105L, Package_TO_SOT_SMD:SOT-23, symbol Power_Protection:NUP2105L
- added D13: 1N5819WS, Diode_SMD:D_SOD-323, symbol Device:D_Schottky
- added D14, D15: SMF6.0A, Diode_SMD:D_SMF, symbol Diode:SMAJ6.0A
- added F1: 100mA, Fuse:Fuse_0603_1608Metric, symbol Device:Polyfuse_Small
- added J10: CAN1, Connector_JST:JST_GH_SM04B-GHS-TB_1x04-1MP_P1.25mm_Horizontal, symbol Connector_Generic_MountingPin:Conn_01x04_MountingPin
- added J11: CAN2, Connector_JST:JST_GH_SM04B-GHS-TB_1x04-1MP_P1.25mm_Horizontal, symbol Connector_Generic_MountingPin:Conn_01x04_MountingPin
- added J5: TELEM1, Connector_JST:JST_GH_SM06B-GHS-TB_1x06-1MP_P1.25mm_Horizontal, symbol Connector_Generic_MountingPin:Conn_01x06_MountingPin
- added J6: TELEM3, Connector_JST:JST_GH_SM06B-GHS-TB_1x06-1MP_P1.25mm_Horizontal, symbol Connector_Generic_MountingPin:Conn_01x06_MountingPin
- added J7: GPS1, Connector_JST:JST_GH_SM10B-GHS-TB_1x10-1MP_P1.25mm_Horizontal, symbol Connector_Generic_MountingPin:Conn_01x10_MountingPin
- added J8: GPS2, Connector_JST:JST_GH_SM06B-GHS-TB_1x06-1MP_P1.25mm_Horizontal, symbol Connector_Generic_MountingPin:Conn_01x06_MountingPin
- added J9: I2C, Connector_JST:JST_GH_SM04B-GHS-TB_1x04-1MP_P1.25mm_Horizontal, symbol Connector_Generic_MountingPin:Conn_01x04_MountingPin
- added Q5: AO3400A, Package_TO_SOT_SMD:SOT-23, symbol Transistor_FET:AO3400A
- added R50, R51, R52, R53, R54, R55, R56, R57, R62, R63, R68: 100, Resistor_SMD:R_0402_1005Metric, symbol Device:R_Small_US
- added R58, R59, R64, R65, R66, R67: 22, Resistor_SMD:R_0402_1005Metric, symbol Device:R_Small_US
- added R60: 1k, Resistor_SMD:R_0402_1005Metric, symbol Device:R_Small_US
- added R61: 220, Resistor_SMD:R_0402_1005Metric, symbol Device:R_Small_US
- added R69: 100k, Resistor_SMD:R_0402_1005Metric, symbol Device:R_Small_US
- added U19, U20, U21, U22, U23: TPD4E05U06DQA, Package_SON:USON-10_2.5x1.0mm_P0.5mm, symbol Power_Protection:TPD4E05U06DQA
Connections:
- new net: Q5.1 (G), R68.2, R69.1
- new net CAN1_H: D11.1 (K), J10.2 (Pin_2)
- new net CAN1_L: D11.2 (K), J10.3 (Pin_3)
- new net CAN2_H: D12.1 (K), J11.2 (Pin_2)
- new net CAN2_L: D12.2 (K), J11.3 (Pin_3)
- new net FMU_BUZZER: R68.1
- new net FMU_I2C1_SCL_GPS1: R58.1
- new net FMU_I2C1_SDA_GPS1: R59.1
- new net FMU_I2C2_SCL_GPS2: R64.1, R66.1
- new net FMU_I2C2_SDA_GPS2: R65.1, R67.1
- new net FMU_UART7_CTS_TEL1: R52.1
- new net FMU_UART7_RTS_TEL1: R53.1
- new net FMU_UART7_RX_TEL1: R51.1
- new net FMU_UART7_TX_TEL1: R50.1
- new net FMU_UART8_RX_GPS2: R63.1
- new net FMU_UART8_TX_GPS2: R62.1
- new net FMU_USART1_RX_GPS1: R57.1
- new net FMU_USART1_TX_GPS1: R56.1
- new net FMU_USART2_RX_TEL3: R55.1
- new net FMU_USART2_TX_TEL3: R54.1
- new net FMU_VDD_3V3: F1.1
- new net FMU_VDD_5V_HIPWR: C57.1, D15.1 (A1), J5.1 (Pin_1), J8.1 (Pin_1)
- new net FMU_VDD_5V_PERIPH: C56.1, D13.1 (K), D14.1 (A1), J10.1 (Pin_1), J11.1 (Pin_1), J6.1 (Pin_1), J7.1 (Pin_1), J9.1 (Pin_1)
- new net GND: C55.2, C56.2, C57.2, D11.3 (A), D12.3 (A), D14.2 (A2), D15.2 (A2), J10.4 (Pin_4), J10.MP (MountPin), J11.4 (Pin_4), J11.MP (MountPin), J5.6 (Pin_6), J5.MP (MountPin), J6.6 (Pin_6), J6.MP (MountPin), J7.10 (Pin_10), J7.MP (MountPin), J8.6 (Pin_6), J8.MP (MountPin), J9.4 (Pin_4), J9.MP (MountPin), Q5.2 (S), R69.2, U19.3 (GND), U19.8 (GND), U20.3 (GND), U20.8 (GND), U21.3 (GND), U21.8 (GND), U22.3 (GND), U22.8 (GND), U23.3 (GND), U23.8 (GND)
- new net GPS1_3V3: C55.1, F1.2, J7.8 (Pin_8)
- new net GPS1_BUZZER: D13.2 (A), J7.9 (Pin_9), Q5.3 (D), U22.4 (D2+)
- new net GPS1_LED: J7.7 (Pin_7), R61.2, U22.2 (D1-)
- new net GPS1_RX: J7.3 (Pin_3), R57.2, U21.2 (D1-)
- new net GPS1_SCL: J7.4 (Pin_4), R58.2, U21.4 (D2+)
- new net GPS1_SDA: J7.5 (Pin_5), R59.2, U21.5 (D2-)
- new net GPS1_SW: J7.6 (Pin_6), R60.2, U22.1 (D1+)
- new net GPS1_TX: J7.2 (Pin_2), R56.2, U21.1 (D1+)
- new net GPS2_RX: J8.3 (Pin_3), R63.2, U23.2 (D1-)
- new net GPS2_SCL: J8.4 (Pin_4), R64.2, U23.4 (D2+)
- new net GPS2_SDA: J8.5 (Pin_5), R65.2, U23.5 (D2-)
- new net GPS2_TX: J8.2 (Pin_2), R62.2, U23.1 (D1+)
- new net I2C_SCL: J9.2 (Pin_2), R66.2, U20.4 (D2+)
- new net I2C_SDA: J9.3 (Pin_3), R67.2, U20.5 (D2-)
- new net IO_SAFETY_SWITCH: R60.1
- new net N_IO_LED_SAFETY: R61.1
- new net TELEM1_CTS: J5.4 (Pin_4), R52.2, U19.4 (D2+)
- new net TELEM1_RTS: J5.5 (Pin_5), R53.2, U19.5 (D2-)
- new net TELEM1_RX: J5.3 (Pin_3), R51.2, U19.2 (D1-)
- new net TELEM1_TX: J5.2 (Pin_2), R50.2, U19.1 (D1+)
- new net TELEM3_RX: J6.3 (Pin_3), R55.2, U20.2 (D1-)
- new net TELEM3_TX: J6.2 (Pin_2), R54.2, U20.1 (D1+)
- no-connect marks 0 -> 23
Other:
- note added: "Buzzer driver"
- note added: "Pixhawk connector standard DS-009, JST-GH 1.25 mm. Pin 1 is VCC on every port. Each signal: connector, ESD array line (port-side net), series resistor, processor. CAN has no series resistors. N_IO_LED_SAFETY: active low, open drain. GPS1 pin 9 (GPS1_BUZZER) is the buzzer low side; FMU_BUZZER high sounds it. All pins have ESD protection for static shock"
- note added: "Rail clamps and GPS1 3.3 V decoupling"
