File: projects/pinion/hardware/pinion-main/sensors.kicad_sch (KiCad schematic)
At the start: 0 parts

Commit message: [pinion] added all the sensors
Parts:
- added U5: IST8310, Package_LGA:LGA-16_3x3mm_P0.5mm, symbol Sensor_Magnetic:IST8310
- added U6: MS5611-01BA, Package_LGA:LGA-8_3x5mm_P1.25mm, symbol Sensor_Pressure:MS5611-01BA
- added U8: ICM-42688-P, Sensors:LGA-14_3x2.5mm_P0.5mm_LayoutBorder3x4y, symbol lib:ICM-42688-P
- added U9: BMI270, Sensors:Bosch_LGA-14_3x2.5mm_P0.5mm, symbol lib:BMI270
Connections:
- new net: U6.4 (CSB), U6.5 (CSB)
- new net: U5.11 (VSS), U5.9 (VSS)

Commit message: [pinion] fmu sensors, external heated sensor board
Parts:
- removed U8: ICM-42688-P, Sensors:LGA-14_3x2.5mm_P0.5mm_LayoutBorder3x4y, symbol lib:ICM-42688-P
- removed U9: BMI270, Sensors:Bosch_LGA-14_3x2.5mm_P0.5mm, symbol lib:BMI270
- added C51, C52, C53: 100n, Capacitor_SMD:C_0402_1005Metric, symbol Device:C_Small
- added C54: 4.7u, Capacitor_SMD:C_0603_1608Metric, symbol Device:C_Small
- added J4: IMU FFC 22, Connector_FFC-FPC:Hirose_FH12-22S-0.5SH_1x22-1MP_P0.50mm_Horizontal, symbol Connector_Generic_MountingPin:Conn_01x22_MountingPin
Connections:
- net FMU_VDD_3V3_SENSORS: now reaches U6.1 (VDD)
- net FMU_VDD_3V3_SENSORS: now also U5.13 (DVDD), U5.14 (~{RST}), U5.2 (AVDD), U6.2 (PS), C51.1, C52.1, C53.1, J4.2 (Pin_2), J4.3 (Pin_3)
- net GND: now reaches U6.3 (GND)
- net GND: now also U5.11 (VSS), U5.5 (CAD0), U5.6 (CAD1), U5.9 (VSS), U6.4 (CSB), U6.5 (CSB), C51.2, C52.2, C53.2, C54.2, J4.1 (Pin_1), J4.14 (Pin_14), J4.17 (Pin_17), J4.22 (Pin_22), J4.4 (Pin_4), J4.6 (Pin_6), J4.9 (Pin_9), J4.MP (MountPin)
- net FMU_I2C4_SDA: now reaches U6.7 (SDI/SDA)
- net FMU_I2C4_SDA: now also U5.16 (SDA), J4.16 (Pin_16)
- net FMU_I2C4_SCL: now reaches U6.8 (SCLK)
- net FMU_I2C4_SCL: now also U5.1 (SCL), J4.15 (Pin_15)
- net at U5.10 (C1): now also C54.1
- new net +5V: J4.20 (Pin_20), J4.21 (Pin_21)
- new net FMU_HEATER: J4.18 (Pin_18)
- new net FMU_SPI1_CS1_BMI270: J4.10 (Pin_10)
- new net FMU_SPI1_CS3_ICM42688: J4.11 (Pin_11)
- new net FMU_SPI1_DRDY1_BMI270: J4.12 (Pin_12)
- new net FMU_SPI1_DRDY3_ICM42688: J4.13 (Pin_13)
- new net FMU_SPI1_MISO_SENSOR: J4.8 (Pin_8)
- new net FMU_SPI1_MOSI_SENSOR: J4.7 (Pin_7)
- new net FMU_SPI1_SCK_SENSOR: J4.5 (Pin_5)
- no-connect marks 0 -> 4
Other:
- note added: "Barometer: MS5611, I2C4 0x77"
- note added: "IMU board connector: 22-way 0.5 mm FFC"
- note added: "Magnetometer: IST8310, I2C4 0x0C"
- moved on the sheet: U5, U6

Commit message: [pinion] fmu connectors and esd protection
Other:
- note added: "ORIENTATION, as on the FMUv6C (top side, seen from above) U5 IST8310: +X forward, +Y to starboard, +Z up. PX4: ist8310, no rotation U6 MS5611: no orientation; keep it away from heat, light and airflow"
Changed lines of the file:
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@@
+		)
+	)
+	(text "ORIENTATION, as on the FMUv6C (top side, seen from above)\nU5 IST8310: +X forward, +Y to starboard, +Z up. PX4: ist8310, no rotation\nU6 MS5611: no orientation; keep it away from heat, light and airflow"
+		(exclude_from_sim no)
+		(at 116.84 127 0)
+		(effects
+			(font
+				(size 1.27 1.27)
+			)
+			(justify left top)
 		)
 	)
