File: projects/pinion/hardware/pinion-main/fmu.kicad_sch (KiCad schematic)
At the start: 0 parts

Commit message: [pinion] mcu basic schematic in
Connections:
- no-connect marks 0 -> 2
Other:
- sheet fmu-power ports: added FMU_VDD_3V3_SENSORS_EN, FMU_VDD_3V3_SENSORS_FLT, FMU_VDD_5V_HIPWR_EN, FMU_VDD_5V_HIPWR_FLT, FMU_VDD_5V_PERIPH_EN, FMU_VDD_5V_PERIPH_FLT, IO_VDD_3V3_SPEKTRUM_EN, IO_VDD_3V3_SPEKTRUM_FLT; removed none
Changed lines of the file:
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@@
 	(generator_version "10.0")
 	(paper "A4")
+	(no_connect
+		(at 93.98 50.8)
+	)
+	(no_connect
+		(at 93.98 57.15)
+	)
 	(sheet
 		(at 104.14 101.6)
@@
 	(sheet
 		(at 59.69 44.45)
-		(size 39.37 26.67)
+		(size 34.29 29.21)
 		(exclude_from_sim no)
 		(in_bom yes)
@@
 		)
 		(property "Sheetfile" "fmu-power.kicad_sch"
-			(at 59.69 71.7046 0)
-			(show_name no)
-			(do_not_autoplace no)
-			(effects
-				(font
-					(size 1.27 1.27)
-				)
-				(justify left top)
-			)
-		)
+			(at 59.69 74.2446 0)
+			(show_name no)
+			(do_not_autoplace no)
+			(effects
+				(font
+					(size 1.27 1.27)
+				)
+				(justify left top)
+			)
+		)
+		(pin "IO_VDD_3V3_SPEKTRUM_EN" input
+			(at 93.98 48.26 0)
+			(effects
+				(font
+					(size 1.27 1.27)
+				)
+				(justify right)
+			)
+		)
+		(pin "FMU_VDD_3V3_SENSORS_FLT" output
+			(at 93.98 57.15 0)
+			(effects
+				(font
+					(size 1.27 1.27)
+				)
+				(justify right)
+			)
+		)
+		(pin "FMU_VDD_5V_HIPWR_EN" input
+			(at 93.98 60.96 0)
+			(effects
+				(font
+					(size 1.27 1.27)
+				)
+				(justify right)
+			)
+		)
+		(pin "IO_VDD_3V3_SPEKTRUM_FLT" output
+			(at 93.98 50.8 0)
+			(effects
+				(font
+					(size 1.27 1.27)
+				)
+				(justify right)
+			)
+		)
+		(pin "FMU_VDD_5V_HIPWR_FLT" output
+			(at 93.98 63.5 0)
+			(effects
+				(font
+					(size 1.27 1.27)
+				)
+				(justify right)
+			)
+		)
+		(pin "FMU_VDD_5V_PERIPH_EN" input
+			(at 93.98 67.31 0)
+			(effects
+				(font
+					(size 1.27 1.27)
+				)
+				(justify right)
+			)
+		)
+		(pin "FMU_VDD_5V_PERIPH_FLT" output
+			(at 93.98 69.85 0)
+			(effects
+				(font
+					(size 1.27 1.27)
+				)
+				(justify right)
+			)
+		)
+		(pin "FMU_VDD_3V3_SENSORS_EN" input
+			(at 93.98 54.61 0)
+			(effects
+				(font
+					(size 1.27 1.27)
+				)
+				(justify right)
+			)
+		)

Commit message: [pinion] fmu can transievers
Other:
- sheet fmu-connectors ports: added CAN1_H, CAN1_L, CAN2_H, CAN2_L, FMU_BUZZER, FMU_I2C1_SCL_GPS1, FMU_I2C1_SDA_GPS1, FMU_I2C2_SCL_GPS2, FMU_I2C2_SDA_GPS2, FMU_UART7_CTS_TEL1, FMU_UART7_RTS_TEL1, FMU_UART7_RX_TEL1, FMU_UART7_TX_TEL1, FMU_UART8_RX_GPS2, FMU_UART8_TX_GPS2, FMU_USART1_RX_GPS1, FMU_USART1_TX_GPS1, FMU_USART2_RX_TEL3, FMU_USART2_TX_TEL3, IO_SAFETY_SWITCH, N_IO_LED_SAFETY; removed none
- sheet sensors ports: added FMU_HEATER, FMU_I2C4_SCL, FMU_I2C4_SDA, FMU_SPI1_CS1_BMI270, FMU_SPI1_CS3_ICM42688, FMU_SPI1_DRDY1_BMI270, FMU_SPI1_DRDY3_ICM42688, FMU_SPI1_MISO_SENSOR, FMU_SPI1_MOSI_SENSOR, FMU_SPI1_SCK_SENSOR; removed none
