File: projects/pinion/hardware/pinion-imu/pinion-imu.kicad_sch (KiCad schematic)
At the start: 24 parts, among them J1 IMU FFC 22, Q1 AO3400A, U1 BMI270, U2 ICM-42688-P, U3 24LC64, U4 LM4040DBZ-2.5, U5 TLV9001IDCK

Commit message: [pinion] fmu connectors and esd protection
Other:
- note added: "ORIENTATION, as on the FMUv6C (parts on the top side, seen from above) U2 ICM-42688-P: +X to port, +Y aft, +Z up; pin 1 at the aft-starboard corner. PX4: icm42688p -R 6 U1 BMI270: +X aft, +Y to starboard, +Z up; pin 1 at the aft-starboard corner. PX4: bmi270 -R 4 Forward is the airframe's forward once this board is mounted."
Changed lines of the file:
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@@
+		)
+	)
+	(text "ORIENTATION, as on the FMUv6C (parts on the top side, seen from above)\nU2 ICM-42688-P: +X to port, +Y aft, +Z up; pin 1 at the aft-starboard corner. PX4: icm42688p -R 6\nU1 BMI270: +X aft, +Y to starboard, +Z up; pin 1 at the aft-starboard corner. PX4: bmi270 -R 4\nForward is the airframe's forward once this board is mounted."
+		(exclude_from_sim no)
+		(at 30.48 86.36 0)
+		(effects
+			(font
+				(size 1.27 1.27)
+			)
+			(justify left top)
 		)
 	)
